Commit message: Fix GPS antenna lever-arm: place base_footprint at front antenna
The EKF estimated base_footprint 0.95 m ahead of true, because the GPS sits at
gps_link (wheelbase/2+0.35 forward) while navsat_transform treats the fix as
base_footprint. navsat's implicit gps_link->base_footprint TF correction does
not apply reliably (and robot_localization exposes no offset parameter), and
solbot4 never corrected it either (its real /gps/fix has empty frame_id).

Fix: define base_footprint to coincide with the front antenna — shift base_joint
(base_footprint->base_link) back by -(wheelbase/2+0.35) so gps_link lands at
base_footprint. The GPS then measures base_footprint directly, zero lever-arm,
consistent sim and real. sim_gps_fix_publisher antenna offset set to 0.

Verified: EKF /odom coincides with /odometry/gazebo — offset 0.00 m stationary,
<=0.07 m through forward + turns (was 0.95 m and growing).

Note: a URDF comment line must not start with "word:" — launch_ros parses the
robot_description string as YAML and a leading key-colon aborts the whole launch
("Unable to parse robot_description as yaml"). Kept the comment single-line.

Co-Authored-By: Claude Opus 4.8 <noreply@anthropic.com>

File: src/solbot5_description/urdf/solbot5_description.urdf (robot description, URDF)
Before this commit: robot solbot5, 5 links, 4 joints
Joints:
- joint base_joint: origin xyz=0.0 0.0 ${(wheel_radius+wheel_zoff)} rpy=0 0 0 -> xyz=${-(wheelbase/2 + 0.35)} 0.0 ${(wheel_radius+wheel_zoff)} rpy=0 0 0
