Commit message: Add tool_link: symmetry line, ground plane, 80cm behind front axle

File: src/description/description/urdf/description.urdf (robot description, URDF)
Before this commit: robot solbot5, 5 links, 4 joints
Links:
- added link tool_link
Joints:
- added joint tool_joint: type fixed, parent base_footprint, child tool_link, origin xyz=-1.35 0.0 0.0 rpy=0 0 0

Commit message: Replace RsPathController with MPC pure-pursuit + segment-aware tracking
Complete rewrite of rs_path_controller for Ackermann robots on RS paths:

Controller:
- MPC-style: simulate Ackermann arc, find intersection with path, binary-search
  steering angle to place cross point at adaptive lookahead distance
- Pure-pursuit steering with CTE correction term for straight-segment tracking
- Adaptive lookahead: clamp(min_look + dist_to_path, min, max)
- Segment-aware closestIndex: caps search within current fwd/reverse segment
  to prevent RS path self-intersection from causing 30+ waypoint index jumps
- segmentEndIndex caps lookahead/arc_end at direction boundaries so PP target
  never crosses fwd/reverse boundary (eliminates max-steer at transitions)
- Goal checker switched to SimpleGoalChecker with yaw tolerance

URDF / sim:
- base_footprint moved to rear axle (Ackermann pivot); base_link 0.40m ahead
- tool_link aliased to base_footprint (zero offset)
- Steering hinge friction 2.0→0.0, damping 0.0→0.5 (eliminates 4s servo lag)
- sim GPS antenna_x corrected to 1.35m (was 0.0)

Logger:
- rs_controller_logger.py updated for new 11-field debug format
- Added ctrl_lookahead and ctrl_dist_to_path columns

File: src/description/description/urdf/description.urdf (robot description, URDF)
Before this commit: robot solbot5, 6 links, 5 joints
Joints:
- joint base_joint: origin xyz=${-(wheelbase/2 + 0.35)} 0.0 ${(wheel_radius+wheel_zoff)} rpy=0 0 0 -> xyz=${wheelbase/2 - wheel_radius} 0.0 ${(wheel_radius+wheel_zoff)} rpy=0 0 0
- joint tool_joint: origin xyz=-1.35 0.0 0.0 rpy=0 0 0 -> xyz=0.0 0.0 0.0 rpy=0 0 0

File: src/description/description/urdf/solbot3_steering_hinge.xacro (robot description, xacro)
@@ -27,5 +27,5 @@
             <axis xyz="0 0 1" />
             <limit lower="-0.523598767" upper="0.523598767" effort="1000" velocity="1.0" />
-            <dynamics damping="0.0" friction="2.0"/>
+            <dynamics damping="0.5" friction="0.0"/>
         </joint>
         <link name="${wheel_prefix}_wheel_link">
@@ -85,5 +85,5 @@
             <axis xyz="0 0 -1"/>
             <limit lower="-0.523598767" upper="0.523598767" effort="1000" velocity="1.0" />
-            <dynamics damping="0.0" friction="2.0"/>
+            <dynamics damping="0.5" friction="0.0"/>
         </joint>
         <link name="front_right_wheel_link">
