Commit message: Fix sim steering: geometry, gains, limits, effective wheelbase
- URDF: remove wheel_radius offset from all 5 joint origins so
  axle-to-axle equals wheelbase (1.20m) as intended
- URDF: fix kingpin_width and wheel_separation to use \${track} (0.77m)
  instead of hardcoded 0.6m
- URDF: add steer_p_gain=100 to AckermannSteering plugin so joints
  track commanded angle at useful speed
- URDF: set wheel_base=1.33 in plugin (measured effective wheelbase)
- URDF: set steering_limit=0.610865 rad (35°) consistently
- Steering hinge xacro: raise joint velocity limit 1→20 rad/s,
  joint angle limit ±30°→±35° to match plugin and controller
- nav2_params_m3: wheelbase 1.20→1.33 (empirical: w_actual/w_expected
  = 0.905 across all arcs, implying L_eff = 1.20/0.905 ≈ 1.33m)
- nav2_params_m3: max_steering_angle 0.7→0.610865 rad (35°)

File: src/description/description/urdf/description.urdf (robot description, URDF)
Before this commit: robot solbot5, 6 links, 5 joints
Joints:
- joint base_joint: origin xyz=${wheelbase/2 - wheel_radius} 0.0 ${(wheel_radius+wheel_zoff)} rpy=0 0 0 -> xyz=${wheelbase/2} 0.0 ${(wheel_radius+wheel_zoff)} rpy=0 0 0

File: src/description/description/urdf/solbot3_steering_hinge.xacro (robot description, xacro)
@@ -26,5 +26,5 @@
             <xacro:insert_block name="joint_pose"/>
             <axis xyz="0 0 1" />
-            <limit lower="-0.523598767" upper="0.523598767" effort="1000" velocity="1.0" />
+            <limit lower="-0.610865" upper="0.610865" effort="1000" velocity="20.0" />
             <dynamics damping="0.5" friction="0.0"/>
         </joint>
@@ -84,5 +84,5 @@
             <xacro:insert_block name="joint_pose"/>
             <axis xyz="0 0 -1"/>
-            <limit lower="-0.523598767" upper="0.523598767" effort="1000" velocity="1.0" />
+            <limit lower="-0.610865" upper="0.610865" effort="1000" velocity="20.0" />
             <dynamics damping="0.5" friction="0.0"/>
         </joint>

Commit message: tool-slider: URDF tool_bar+OAK-D, PauseProgressChecker, rviz_m4, sim fixes
- Add tool_bar link (0.8m sliding toolbar) and oakd_link (OAK-D Lite camera)
  to URDF with Gazebo RGBD sensor on /oakd/rgb
- Add simulation.launch.py ParameterValue fix for xacro with negative expressions
- Add PauseProgressChecker plugin: pauses nav instead of cancelling goal on stall
- Switch nav2_params_m3 progress_checker to PauseProgressChecker
- Update pause guard in field_nav_sim.xml to save field progress before waiting
- Add rviz_m4.rviz config and run_rviz_m4.sh
- unset LD_LIBRARY_PATH in run_field_sim.sh and run_m3_sim.sh

File: src/description/description/urdf/description.urdf (robot description, URDF)
Before this commit: robot solbot5, 6 links, 5 joints
Links:
- added link oakd_link, mass 0.061; collision box size=0.036 0.091 0.028; visual box size=0.036 0.091 0.028
- added link oakd_rgb_optical_frame
- added link tool_bar, mass 3.0; collision box size=0.05 0.80 0.05; visual box size=0.05 0.80 0.05
Joints:
- added joint oakd_joint: type fixed, parent base_footprint, child oakd_link, origin xyz=0.0 0.0 0.50 rpy=0 ${-M_PI/2} 0
- added joint oakd_rgb_optical_joint: type fixed, parent oakd_link, child oakd_rgb_optical_frame, origin xyz=0 0 0 rpy=${-M_PI/2} 0 ${-M_PI/2}
- added joint tool_bar_joint: type fixed, parent tool_link, child tool_bar, origin xyz=0.0 0.0 0.0 rpy=0 0 0

Commit message: URDF: add 3 implements on tool_bar; move toolbar+camera 0.5m fwd 0.4m up
- tool_bar_joint: xyz 0→0.5m forward, 0→0.4m up (relative to tool_link)
- oakd_joint: xyz 0→0.5m forward, 0.50→0.90m up (relative to base_footprint)
- Add 3 red implement links (10×2×10cm) on tool_bar: center + ±36cm lateral,
  20cm behind tool_bar centre
- tool_actuator_sim: TF x=0.5 z=0.4 to match URDF tool_bar offset

File: src/description/description/urdf/description.urdf (robot description, URDF)
Before this commit: robot solbot5, 9 links, 8 joints
Links:
- added link implement_center, mass 0.5; collision box size=0.10 0.02 0.10; visual box size=0.10 0.02 0.10
- added link implement_left, mass 0.5; collision box size=0.10 0.02 0.10; visual box size=0.10 0.02 0.10
- added link implement_right, mass 0.5; collision box size=0.10 0.02 0.10; visual box size=0.10 0.02 0.10
Joints:
- added joint implement_center_joint: type fixed, parent tool_bar, child implement_center, origin xyz=-0.20 0.0 0.0 rpy=0 0 0
- added joint implement_left_joint: type fixed, parent tool_bar, child implement_left, origin xyz=-0.20 0.36 0.0 rpy=0 0 0
- added joint implement_right_joint: type fixed, parent tool_bar, child implement_right, origin xyz=-0.20 -0.36 0.0 rpy=0 0 0
- joint oakd_joint: origin xyz=0.0 0.0 0.50 rpy=0 ${-M_PI/2} 0 -> xyz=0.5 0.0 0.90 rpy=0 ${-M_PI/2} 0
- joint tool_bar_joint: origin xyz=0.0 0.0 0.0 rpy=0 0 0 -> xyz=0.5 0.0 0.4 rpy=0 0 0

Commit message: tool-slider: prismatic tool_bar_joint, camera fix, web_video_server
- tool_bar_joint: fixed→prismatic (y-axis ±10cm), driven by JointPositionController
- tool_actuator_sim: publish Float64 to /tool_bar_joint/cmd_pos instead of TF
- gz_bridge: add tool_bar_joint/cmd_pos (ROS→GZ) and oakd camera topics (GZ→ROS)
- oakd_joint: fix pitch to M_PI/2 (was -M_PI/2, was looking up not down)
- oakd_joint: lower camera 10cm to z=0.80m
- tool_bar_joint: move 10cm forward to x=0.6m
- implements: resize to 3x2x1cm, move 20cm back on tool_bar
- m4_nav_sim: add web_video_server node on port 8080

File: src/description/description/urdf/description.urdf (robot description, URDF)
Before this commit: robot solbot5, 12 links, 11 joints
Links:
- link implement_center: geometry collision box size=0.03 0.02 0.01; visual box size=0.03 0.02 0.01
- link implement_left: geometry collision box size=0.03 0.02 0.01; visual box size=0.03 0.02 0.01
- link implement_right: geometry collision box size=0.03 0.02 0.01; visual box size=0.03 0.02 0.01
Joints:
- joint oakd_joint: origin xyz=0.5 0.0 0.90 rpy=0 ${-M_PI/2} 0 -> xyz=0.5 0.0 0.80 rpy=0 ${M_PI/2} 0
- joint tool_bar_joint: axis (none) -> 0 1 0; limit (none) -> lower=-0.10 upper=0.10 effort=100 velocity=0.5; origin xyz=0.5 0.0 0.4 rpy=0 0 0 -> xyz=0.6 0.0 0.4 rpy=0 0 0; type fixed -> prismatic

Commit message: temp: remove toolbar and implements from URDF for QR localization testing
The toolbar (tool_bar link at z=0.4m forward of tool_link) bisects the
downward camera image, occluding QR codes in the centre row and dropping
the decode rate. Removing it gives the camera an unobstructed floor view.

Also removes:
- tool_bar_joint from JointStatePublisher plugin
- JointPositionController plugin for tool_bar_joint

Restore with: git checkout HEAD~1 -- src/description/description/urdf/description.urdf

File: src/description/description/urdf/description.urdf (robot description, URDF)
Before this commit: robot solbot5, 12 links, 11 joints
Links:
- removed link implement_center
- removed link implement_left
- removed link implement_right
- removed link tool_bar
Joints:
- removed joint implement_center_joint
- removed joint implement_left_joint
- removed joint implement_right_joint
- removed joint tool_bar_joint

Commit message: feat: re-enable toolbar, green crop rows, remove QR floor, add M5 script
- Restore tool_bar/tool_bar_joint/implement_* in URDF (removed in 6413f52
  for QR-decode camera testing, no longer needed since the QR floor is gone).
- Remove qr_floor model from house_short_rows.sdf (dormant, no active
  launch path used grid_decoder.py against it).
- crop_row_spawner: render all segments green instead of the 8-color
  debug cycle.
- Add run_m5_field_sim.sh (copy of run_m4_field_sim.sh, logs to
  logs/m5_field_sim/) with a rolling crop_row_spawner instance so a row
  segment is always spawned ahead of the robot and removed once passed.

File: src/description/description/urdf/description.urdf (robot description, URDF)
Before this commit: robot solbot5, 8 links, 7 joints
Links:
- added link implement_center, mass 0.5; collision box size=0.03 0.02 0.01; visual box size=0.03 0.02 0.01
- added link implement_left, mass 0.5; collision box size=0.03 0.02 0.01; visual box size=0.03 0.02 0.01
- added link implement_right, mass 0.5; collision box size=0.03 0.02 0.01; visual box size=0.03 0.02 0.01
- added link tool_bar, mass 3.0; collision box size=0.05 0.80 0.05; visual box size=0.05 0.80 0.05
Joints:
- added joint implement_center_joint: type fixed, parent tool_bar, child implement_center, origin xyz=-0.20 0.0 0.0 rpy=0 0 0
- added joint implement_left_joint: type fixed, parent tool_bar, child implement_left, origin xyz=-0.20 0.36 0.0 rpy=0 0 0
- added joint implement_right_joint: type fixed, parent tool_bar, child implement_right, origin xyz=-0.20 -0.36 0.0 rpy=0 0 0
- added joint tool_bar_joint: type prismatic, parent tool_link, child tool_bar, origin xyz=0.6 0.0 0.4 rpy=0 0 0, axis 0 1 0, limit lower=-0.10 upper=0.10 effort=100 velocity=0.5
